File: Switch-Ethernet/Rev A4/SwitchEthernet - Rev A4.sch (EAGLE design)
At the start: 118 parts, among them J1 22-05-7028-02, J2 DF17(4.0)-20DS-0.5V(57), J3 DF17(4.0)-20DP-0.5V(57), P1 RB1-125BAG1A, T1 H1102FNL, T2 H1102FNL, T3 EXMACHINA-LOGO-NAME, U1 TC1264-3.3, U2 TC1264-1.8, U3 KSZ8995MA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

Commit message: Place name and value correctly on the board
Parts:
- removed -25.000MHZMAAJ-T1: 8Z-25.000MHZMAAJ-T, crystal:8Z-25.000MHZMAAJ-T
- removed CR1: SMAJ33A-E3/61, diode:SMAJ33A-E3/61
- removed X2: NE8FAV, con-neutrik_ag:NE8FAV
- added D2: 1N4148WS, diode:1N4148WS
- added J4: DF17(4.0)-20DS-0.5V(57), con-hirose:DF17(4.0)-20DS-0.5V(57)
- added J5: DF17(4.0)-20DP-0.5V(57), con-hirose:DF17(4.0)-20DP-0.5V(57)
- D1: value 1N4148WS -> SMAJ33A-E3/61; device diode:1N4148WS -> diode:SMAJ33A-E3/61; MF (none) -> VISHAY; MPN (none) -> SMAJ33A-E3/5A; OC_FARNELL unknown -> 1812505; OC_NEWARK 01P4213 -> 08R3790
- J2: value DF17(4.0)-20DS-0.5V(57) -> NE8FAV; device con-hirose:DF17(4.0)-20DS-0.5V(57) -> con-neutrik_ag:NE8FAV; OC_FARNELL (none) -> 1202031; OC_NEWARK (none) -> 01M8373
- J3: value DF17(4.0)-20DP-0.5V(57) -> NE8FAV; device con-hirose:DF17(4.0)-20DP-0.5V(57) -> con-neutrik_ag:NE8FAV; OC_FARNELL (none) -> 1202031; OC_NEWARK (none) -> 01M8373
- X1: value NE8FAV -> 8Z-25.000MHZMAAJ-T; device con-neutrik_ag:NE8FAV -> crystal:8Z-25.000MHZMAAJ-T; MF (none) -> TXC; MPN (none) -> 8Z-25.000MAAJ-T; OC_FARNELL 1202031 -> 1842189; OC_NEWARK 01M8373 -> 84R5794
- renumbered P1 to J6
Connections:
- net +3V3: now also D2.1, J4-1.P, J5-1.P; no longer D1.1, J2-1.P, J3-1.P
- net AGND: now also J2.G, J3.G; no longer X1.G, X2.G
- net CT_1: now also J4-10.P, J5-10.P; no longer J2-10.P, J3-10.P
- net CT_2: now also J4-11.P, J5-11.P; no longer J2-11.P, J3-11.P
- net GND: now also D1.A, J4-20.P, J5-20.P, X1.2; no longer -25.000MHZMAAJ-T1.2, CR1.A, J2-20.P, J3-20.P
- net L1-1: now also J4-8.P, J5-8.P; no longer J2-8.P, J3-8.P
- net L1-2: now also J4-9.P, J5-9.P; no longer J2-9.P, J3-9.P
- net L2-1: now also J4-18.P, J5-18.P; no longer J2-18.P, J3-18.P
- net L2-2: now also J4-19.P, J5-19.P; no longer J2-19.P, J3-19.P
- net N$11: now also J2.5; no longer X1.5
- net N$12: now also J3.7; no longer X2.7
- net N$15: now also J3.4; no longer X2.4
- net N$18: now also J3.5; no longer X2.5
- net N$5: now also J3.8; no longer X2.8
- net N$7: now also J2.4; no longer X1.4
- net N$8: now also J2.8; no longer X1.8
- net N$9: now also J2.7; no longer X1.7
- net PW: now also D1.C; no longer CR1.C
- net RST_N: now also D2.2; no longer D1.2
- net RX1_N: now also J2.2, J4-3.P, J5-3.P; no longer J2-3.P, J3-3.P, X1.2
- net RX1_P: now also J2.1, J4-2.P, J5-2.P; no longer J2-2.P, J3-2.P, X1.1
- net RX2_N: now also J3.2, J4-13.P, J5-13.P; no longer J2-13.P, J3-13.P, X2.2
- net RX2_P: now also J3.1, J4-12.P, J5-12.P; no longer J2-12.P, J3-12.P, X2.1
- net TX1_N: now also J2.6, J4-6.P, J5-6.P; no longer J2-6.P, J3-6.P, X1.6
- net TX1_P: now also J2.3, J4-5.P, J5-5.P; no longer J2-5.P, J3-5.P, X1.3
- net TX2_N: now also J3.6, J4-16.P, J5-16.P; no longer J2-16.P, J3-16.P, X2.6
- net TX2_P: now also J3.3, J4-15.P, J5-15.P; no longer J2-15.P, J3-15.P, X2.3
- net X1: now also X1.1; no longer -25.000MHZMAAJ-T1.1
- net X2: now also X1.3; no longer -25.000MHZMAAJ-T1.3

Commit message: Generate MDP
Parts:
- C1, C2, C5, C6: MPN (none) -> MC1206B102K202CT
- C10, C11, C12, C9: MPN (none) -> MC0603B105K160CT; OC_NEWARK (none) -> 06X6171
- C13, C14, C19: MPN (none) -> MCCTA475M010
- C15, C16, C17, C18, C20, C21, C25, C26, C27, C28, C29, C30, C31, C32, C33, C34, C35, C36, C37, C38, C39, C4, C8: MF MULTICOMP -> (none); MPN MC0603B104K250CT -> MC0603B104K160CT
- C22, C24: MF MULTICOMP -> (none); MPN MC0603B183K160CT -> MC0603N180J500CT
- C23, C3, C7: MF MURATA -> (none); MPN GRM32DR71C106KA01L -> MCNP16V106M5X11
- D1: MF VISHAY -> (none); MPN SMAJ33A-E3/5A -> SMAJ33A-E3/61
- D2: MPN (none) -> 1N4148W
- F1: MPN (none) -> 1812L110/24DR; OC_NEWARK (none) -> 39X0319
- J1: MF MOLEX -> (none)
- J4: MPN (none) -> DF17(4.0)-20DS-0.5V(57); OC_NEWARK (none) -> 69W0567
- J5: MPN (none) -> DF17(4.0)-20DP-0.5V(57); OC_NEWARK (none) -> 69W0566
- JP1, JP2, JP3, JP4, MP1, MP2, MP3, MP4, TP1, TP2, TP3, TP4, TP5: OC_NEWARK (none) -> unknown
- L1: MPN (none) -> LQH43CN150K03L
- LED1, LED2, LED3, LED4, LED5, R16, R17, R18, R19: MF MULTICOMP -> (none)
- R1, R10, R11, R12, R13, R2, R4, R5, R6, R7, R8, R9: MF MULTICOMP -> Multicomp Passives; MPN MCMR06X49R9FTL -> MC0063W0603151R
- R14, R15: MF MULTICOMP -> Multicomp Passives; MPN MCMR06X75R0FTL -> MC0063W0603175R
- R20, R21, R22, R23, R24, R25, R26, R27, R30, R31, R32, R33: MF MULTICOMP -> (none); MPN MCMR06X49R9FTL -> MC0603SAF499JT5E
- R28, R29: MF MULTICOMP -> Multicomp Passives; MPN MCMR06X2200FTL -> MC0063W06031220R
- R3: MF MULTICOMP -> Multicomp Passives; MPN MCMR06X1501FTL -> MC0063W060311K5
- R34: MF MULTICOMP -> Multicomp Passives; MPN MCMR06X1002FTL -> MC0063W0603110K
- R35: MF MULTICOMP -> (none); MPN MCMR06X3001FTL -> MC0063W060313K01
- R36, R37: MF (none) -> Multicomp Passives; MPN (none) -> MC0063W0603110K
- R38, R39, R40, R41, R42, R43: MF (none) -> Multicomp Passives; MPN (none) -> MC0603WG00000T5E-TC
- U1: MF (none) -> MICROCHIP; MPN (none) -> TC1264-3.3VAB; OC_NEWARK (none) -> 92C5792
- U2: MF (none) -> MICROCHIP; MPN (none) -> TC1264-1.8VAB; OC_NEWARK (none) -> 92C5783
- U3: MF MICROCHIP -> (none); OC_NEWARK 70Y9044 -> 10AC7950
- U4: MF ATMEL -> (none)
- X1: MF TXC -> (none)

Commit message: Replace device name on D2 and C3, C7, C19
Parts:
- C23, C3, C7: MPN MCNP16V106M5X11 -> GRM188R60J106ME47D; OC_NEWARK 13M5149 -> 24R6334
- D2: MPN 1N4148W -> 1N4148WS.; OC_NEWARK 01P4213 -> 74M5710
Changed lines of the file:
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@@
 <part name="C3" library="rcl" deviceset="C-EU" device="C0603" value="10uF">
 <attribute name="MF" value=""/>
-<attribute name="MPN" value="MCNP16V106M5X11"/>
+<attribute name="MPN" value="GRM188R60J106ME47D"/>
 <attribute name="OC_FARNELL" value="2494299"/>
-<attribute name="OC_NEWARK" value="13M5149"/>
+<attribute name="OC_NEWARK" value="24R6334"/>
 </part>
 <part name="C4" library="rcl" deviceset="C-EU" device="C0603" value="0.1uF">
@@
 <part name="C7" library="rcl" deviceset="C-EU" device="C0603" value="10uF">
 <attribute name="MF" value=""/>
-<attribute name="MPN" value="MCNP16V106M5X11"/>
+<attribute name="MPN" value="GRM188R60J106ME47D"/>
 <attribute name="OC_FARNELL" value="2494299"/>
-<attribute name="OC_NEWARK" value="13M5149"/>
+<attribute name="OC_NEWARK" value="24R6334"/>
 </part>
 <part name="C8" library="rcl" deviceset="C-EU" device="C0603" value="0.1uF">
@@
 <part name="C23" library="rcl" deviceset="C-EU" device="C0603" value="10uF">
 <attribute name="MF" value=""/>
-<attribute name="MPN" value="MCNP16V106M5X11"/>
+<attribute name="MPN" value="GRM188R60J106ME47D"/>
 <attribute name="OC_FARNELL" value="2494299"/>
-<attribute name="OC_NEWARK" value="13M5149"/>
+<attribute name="OC_NEWARK" value="24R6334"/>
 </part>
 <part name="GND22" library="supply1" deviceset="GND" device=""/>
@@
 <part name="D2" library="diode" deviceset="1N4148WS" device="">
 <attribute name="MF" value=""/>
-<attribute name="MPN" value="1N4148W"/>
-<attribute name="OC_FARNELL" value="unknown"/>
-<attribute name="OC_NEWARK" value="01P4213"/>
+<attribute name="MPN" value="1N4148WS."/>
+<attribute name="OC_FARNELL" value="unknown"/>
+<attribute name="OC_NEWARK" value="74M5710"/>
 </part>
 <part name="C1" library="rcl" deviceset="C-EU" device="C1206" value="1000pF, 2kV">

Commit message: Update BOM
Parts:
- D1: MPN SMAJ33A-E3/61 -> (none); OC_NEWARK 08R3790 -> unknown
- U1: MPN TC1264-3.3VAB -> TC1264-3.3VDB; OC_NEWARK 92C5792 -> unknown
- U2: MPN TC1264-1.8VAB -> TC1264-1.8VDBTR; OC_NEWARK 92C5783 -> 92C5784
- U3: MPN KSZ8995MA -> (none); OC_NEWARK 10AC7950 -> unknown
Changed lines of the file:
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@@
 <grid distance="0.1" unitdist="inch" unit="inch" style="lines" multiple="1" display="no" altdistance="0.01" altunitdist="inch" altunit="inch"/>
 <layers>
-<layer number="1" name="Top" color="4" fill="1" visible="no" active="no"/>
-<layer number="2" name="Route2" color="1" fill="3" visible="no" active="no"/>
+<layer number="1" name="Top" color="16" fill="1" visible="no" active="no"/>
+<layer number="2" name="Route2" color="17" fill="1" visible="no" active="no"/>
 <layer number="3" name="Route3" color="4" fill="3" visible="no" active="no"/>
 <layer number="14" name="Route14" color="1" fill="6" visible="no" active="no"/>
-<layer number="15" name="Route15" color="4" fill="6" visible="no" active="no"/>
-<layer number="16" name="Bottom" color="1" fill="1" visible="no" active="no"/>
-<layer number="17" name="Pads" color="2" fill="1" visible="no" active="no"/>
-<layer number="18" name="Vias" color="2" fill="1" visible="no" active="no"/>
+<layer number="15" name="Route15" color="19" fill="1" visible="no" active="no"/>
+<layer number="16" name="Bottom" color="21" fill="1" visible="no" active="no"/>
+<layer number="17" name="Pads" color="18" fill="1" visible="no" active="no"/>
+<layer number="18" name="Vias" color="38" fill="1" visible="no" active="no"/>
 <layer number="19" name="Unrouted" color="6" fill="1" visible="no" active="no"/>
-<layer number="20" name="Dimension" color="15" fill="1" visible="no" active="no"/>
-<layer number="21" name="tPlace" color="7" fill="1" visible="no" active="no"/>
-<layer number="22" name="bPlace" color="7" fill="1" visible="no" active="no"/>
+<layer number="20" name="Dimension" color="7" fill="1" visible="no" active="no"/>
+<layer number="21" name="tPlace" color="55" fill="1" visible="no" active="no"/>
+<layer number="22" name="bPlace" color="54" fill="1" visible="no" active="no"/>
 <layer number="23" name="tOrigins" color="15" fill="1" visible="no" active="no"/>
 <layer number="24" name="bOrigins" color="15" fill="1" visible="no" active="no"/>
-<layer number="25" name="tNames" color="7" fill="1" visible="no" active="no"/>
-<layer number="26" name="bNames" color="7" fill="1" visible="no" active="no"/>
-<layer number="27" name="tValues" color="7" fill="1" visible="no" active="no"/>
-<layer number="28" name="bValues" color="7" fill="1" visible="no" active="no"/>
+<layer number="25" name="tNames" color="55" fill="1" visible="no" active="no"/>
+<layer number="26" name="bNames" color="54" fill="1" visible="no" active="no"/>
+<layer number="27" name="tValues" color="53" fill="1" visible="no" active="no"/>
+<layer number="28" name="bValues" color="52" fill="1" visible="no" active="no"/>
 <layer number="29" name="tStop" color="7" fill="3" visible="no" active="no"/>
 <layer number="30" name="bStop" color="7" fill="6" visible="no" active="no"/>
@@
 <layer number="37" name="tTest" color="7" fill="1" visible="no" active="no"/>
 <layer number="38" name="bTest" color="7" fill="1" visible="no" active="no"/>
-<layer number="39" name="tKeepout" color="4" fill="11" visible="no" active="no"/>
-<layer number="40" name="bKeepout" color="1" fill="11" visible="no" active="no"/>
+<layer number="39" name="tKeepout" color="4" fill="1" visible="no" active="no"/>
+<layer number="40" name="bKeepout" color="3" fill="1" visible="no" active="no"/>
 <layer number="41" name="tRestrict" color="4" fill="10" visible="no" active="no"/>
-<layer number="42" name="bRestrict" color="1" fill="10" visible="no" active="no"/>
+<layer number="42" name="bRestrict" color="3" fill="10" visible="no" active="no"/>
 <layer number="43" name="vRestrict" color="2" fill="10" visible="no" active="no"/>
-<layer number="44" name="Drills" color="7" fill="1" visible="no" active="no"/>
-<layer number="45" name="Holes" color="7" fill="1" visible="no" active="no"/>
-<layer number="46" name="Milling" color="3" fill="1" visible="no" active="no"/>
-<layer number="47" name="Measures" color="7" fill="1" visible="no" active="no"/>
-<layer number="48" name="Document" color="7" fill="1" visible="no" active="no"/>
-<layer number="49" name="Reference" color="7" fill="1" visible="no" active="no"/>
+<layer number="44" name="Drills" color="16" fill="1" visible="no" active="no"/>
+<layer number="45" name="Holes" color="35" fill="1" visible="no" active="no"/>
+<layer number="46" name="Milling" color="35" fill="1" visible="no" active="no"/>
+<layer number="47" name="Measures" color="21" fill="1" visible="no" active="no"/>
+<layer number="48" name="Document" color="24" fill="1" visible="no" active="no"/>
+<layer number="49" name="Reference" color="48" fill="1" visible="no" active="no"/>
 <layer number="50" name="dxf" color="7" fill="1" visible="no" active="no"/>
-<layer number="51" name="tDocu" color="7" fill="1" visible="no" active="no"/>
-<layer number="52" name="bDocu" color="7" fill="1" visible="no" active="no"/>
+<layer number="51" name="tDocu" color="55" fill="1" visible="no" active="no"/>
+<layer number="52" name="bDocu" color="54" fill="1" visible="no" active="no"/>
 <layer number="53" name="tGND_GNDA" color="7" fill="1" visible="no" active="no"/>
 <layer number="54" name="bGND_GNDA" color="7" fill="1" visible="no" active="no"/>
@@
 <part name="D1" library="diode" deviceset="SMAJ33A-E3/61" device="">
 <attribute name="MF" value=""/>
-<attribute name="MPN" value="SMAJ33A-E3/61"/>
+<attribute name="MPN" value=""/>
 <attribute name="OC_FARNELL" value="1812505"/>
-<attribute name="OC_NEWARK" value="08R3790"/>
+<attribute name="OC_NEWARK" value="unknown"/>
 </part>
 <part name="P+2" library="supply1" deviceset="+5V" device=""/>
@@
 <part name="U3" library="Micrel_By_element14_Batch_1" deviceset="KSZ8995MA" device="">
 <attribute name="MF" value=""/>
-<attribute name="MPN" value="KSZ8995MA"/>
+<attribute name="MPN" value=""/>
 <attribute name="OC_FARNELL" value="2509844"/>
-<attribute name="OC_NEWARK" value="10AC7950"/>
+<attribute name="OC_NEWARK" value="unknown"/>
 </part>
 <part name="GND25" library="supply1" deviceset="GND" device=""/>
@@
 <part name="U1" library="microchip-6" deviceset="TC1264-3.3" device="">
 <attribute name="MF" value="MICROCHIP"/>
-<attribute name="MPN" value="TC1264-3.3VAB"/>
-<attribute name="OC_FARNELL" value="unknown"/>
-<attribute name="OC_NEWARK" value="92C5792"/>
+<attribute name="MPN" value="TC1264-3.3VDB"/>
+<attribute name="OC_FARNELL" value="unknown"/>
+<attribute name="OC_NEWARK" value="unknown"/>
 </part>
 <part name="U2" library="microchip-6" deviceset="TC1264-1.8" device="">
 <attribute name="MF" value="MICROCHIP"/>
-<attribute name="MPN" value="TC1264-1.8VAB"/>
-<attribute name="OC_FARNELL" value="unknown"/>
-<attribute name="OC_NEWARK" value="92C5783"/>
+<attribute name="MPN" value="TC1264-1.8VDBTR"/>
+<attribute name="OC_FARNELL" value="unknown"/>
+<attribute name="OC_NEWARK" value="92C5784"/>
 </part>
 <part name="GND8" library="supply1" deviceset="GND" device=""/>
