File: EXM Relay Three/Rev A1/EXM Relay One - Rev A1.brd (EAGLE design)
At the start: 80 x 50 mm, 24 parts, among them J1 MSTBA3, J10 MSTBA2, J2 MSTBA3, J3 22-05-7038-03, J4 22-05-7038-03, J5 22-05-7038-03, J6 22-05-7038-03, J7 MSTBA3, J8 22-05-7038-03, J9 22-05-7038-03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

Commit message: Update relay device and re-route the board
Connections:
- net SIG1_1_NC: now also K1.4; no longer K1.8
- net SIG1_1_NO: now also K1.8; no longer K1.4
- net SIG1_2_NC: now also K1.1; no longer K1.5
- net SIG1_2_NO: now also K1.5; no longer K1.1
- net SIG2_1_NC: now also K2.4; no longer K2.8
- net SIG2_1_NO: now also K2.8; no longer K2.4
- net SIG2_2_NC: now also K2.1; no longer K2.5
- net SIG2_2_NO: now also K2.5; no longer K2.1
- net SIG3_1_NC: now also K3.4; no longer K3.8
- net SIG3_1_NO: now also K3.8; no longer K3.4
- net SIG3_2_NC: now also K3.1; no longer K3.5
- net SIG3_2_NO: now also K3.5; no longer K3.1
Routing:
- net SIG3_2_NO: track 11.0 -> 22.8 mm
- net SIG1_2_NO: track 11.8 -> 23.7 mm
- net SIG2_2_NO: track 11.0 -> 22.2 mm
- net SIG2_1_NC: track 18.4 -> 10.4 mm
- net SIG3_1_NC: track 18.4 -> 10.4 mm
- net SIG1_1_NO: track 10.6 -> 18.4 mm
- net SIG1_1_NC: track 17.6 -> 11.1 mm
- net SIG2_1_NO: track 12.2 -> 17.6 mm
- net SIG3_1_NO: track 12.2 -> 17.0 mm
- net SIG3_2_NC: track 17.4 -> 13.4 mm
- net SIG2_2_NC: track 17.4 -> 13.4 mm
- net SIG1_2_NC: track 18.8 -> 15.4 mm
Changed lines of the file:
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@@
 <signal name="SIG2_1_NO">
 <contactref element="J5" pad="2"/>
-<contactref element="K2" pad="4"/>
+<contactref element="K2" pad="8"/>
 <wire x1="44" y1="5" x2="44" y2="14" width="0.8128" layer="1"/>
-<wire x1="44" y1="14" x2="45.325" y2="15.325" width="0.8128" layer="1"/>
-<wire x1="45.325" y1="15.325" x2="46.605" y2="15.325" width="0.8128" layer="1"/>
+<wire x1="44" y1="14" x2="43" y2="15" width="0.8128" layer="1"/>
+<wire x1="43" y1="15" x2="43" y2="18" width="0.8128" layer="1"/>
+<wire x1="43" y1="18" x2="44.425" y2="19.425" width="0.8128" layer="1"/>
+<wire x1="44.425" y1="19.425" x2="46.605" y2="19.425" width="0.8128" layer="1"/>
 </signal>
 <signal name="SIG1_1_NC">
 <contactref element="J4" pad="1"/>
-<contactref element="K1" pad="8"/>
-<wire x1="21.605" y1="19.425" x2="23.575" y2="19.425" width="0.8128" layer="1"/>
-<wire x1="23.575" y1="19.425" x2="25" y2="18" width="0.8128" layer="1"/>
-<wire x1="25" y1="18" x2="25" y2="9" width="0.8128" layer="1"/>
-<wire x1="25" y1="9" x2="23.54" y2="7.54" width="0.8128" layer="1"/>
-<wire x1="23.54" y1="7.54" x2="23.54" y2="5" width="0.8128" layer="1"/>
+<contactref element="K1" pad="4"/>
+<wire x1="23.54" y1="5" x2="23.54" y2="13.39" width="0.8128" layer="1"/>
+<wire x1="23.54" y1="13.39" x2="21.605" y2="15.325" width="0.8128" layer="1"/>
 </signal>
 <signal name="SIG2_2_NC">
-<contactref element="K2" pad="5"/>
 <contactref element="J6" pad="1"/>
-<wire x1="37.54" y1="5" x2="37.54" y2="17.46" width="0.8128" layer="1"/>
-<wire x1="37.54" y1="17.46" x2="35.575" y2="19.425" width="0.8128" layer="1"/>
-<wire x1="35.575" y1="19.425" x2="33.405" y2="19.425" width="0.8128" layer="1"/>
+<contactref element="K2" pad="1"/>
+<wire x1="37.54" y1="5" x2="37.54" y2="13.46" width="0.8128" layer="1"/>
+<wire x1="37.54" y1="13.46" x2="35.675" y2="15.325" width="0.8128" layer="1"/>
+<wire x1="35.675" y1="15.325" x2="33.405" y2="15.325" width="0.8128" layer="1"/>
 </signal>
 <signal name="SIG2_2_NO">
-<contactref element="K2" pad="1"/>
 <contactref element="J6" pad="2"/>
-<wire x1="35" y1="5" x2="35" y2="13.73" width="0.8128" layer="1"/>
-<wire x1="35" y1="13.73" x2="33.405" y2="15.325" width="0.8128" layer="1"/>
+<contactref element="K2" pad="5"/>
+<wire x1="33.405" y1="19.425" x2="30.425" y2="19.425" width="0.8128" layer="1"/>
+<wire x1="30.425" y1="19.425" x2="29" y2="18" width="0.8128" layer="1"/>
+<wire x1="29" y1="18" x2="29" y2="12" width="0.8128" layer="1"/>
+<wire x1="29" y1="12" x2="31" y2="10" width="0.8128" layer="1"/>
+<wire x1="31" y1="10" x2="34" y2="10" width="0.8128" layer="1"/>
+<wire x1="34" y1="10" x2="35" y2="9" width="0.8128" layer="1"/>
+<wire x1="35" y1="9" x2="35" y2="5" width="0.8128" layer="1"/>
 </signal>
 <signal name="SIG2_1_NC">
 <contactref element="J5" pad="1"/>
-<contactref element="K2" pad="8"/>
-<wire x1="46.54" y1="5" x2="46.54" y2="10.54" width="0.8128" layer="1"/>
-<wire x1="46.54" y1="10.54" x2="50" y2="14" width="0.8128" layer="1"/>
-<wire x1="50" y1="14" x2="50" y2="18" width="0.8128" layer="1"/>
-<wire x1="50" y1="18" x2="48.575" y2="19.425" width="0.8128" layer="1"/>
-<wire x1="48.575" y1="19.425" x2="46.605" y2="19.425" width="0.8128" layer="1"/>
+<contactref element="K2" pad="4"/>
+<wire x1="46.605" y1="15.325" x2="46.54" y2="15.26" width="0.8128" layer="1"/>
+<wire x1="46.54" y1="15.26" x2="46.54" y2="5" width="0.8128" layer="1"/>
 </signal>
 <signal name="SIG_IN_1">
@@
 </signal>
 <signal name="SIG1_1_NO">
-<contactref element="K1" pad="4"/>
 <contactref element="J4" pad="2"/>
-<wire x1="21" y1="5" x2="21" y2="14.72" width="0.8128" layer="1"/>
-<wire x1="21" y1="14.72" x2="21.605" y2="15.325" width="0.8128" layer="1"/>
+<contactref element="K1" pad="8"/>
+<wire x1="21" y1="5" x2="21" y2="9" width="0.8128" layer="1"/>
+<wire x1="21" y1="9" x2="18" y2="12" width="0.8128" layer="1"/>
+<wire x1="18" y1="12" x2="18" y2="18" width="0.8128" layer="1"/>
+<wire x1="18" y1="18" x2="19.425" y2="19.425" width="0.8128" layer="1"/>
+<wire x1="19.425" y1="19.425" x2="21.605" y2="19.425" width="0.8128" layer="1"/>
 </signal>
 <signal name="SIG1_2_NO">
 <contactref element="J3" pad="2"/>
-<contactref element="K1" pad="1"/>
+<contactref element="K1" pad="5"/>
 <wire x1="12" y1="5" x2="12" y2="9" width="0.8128" layer="1"/>
-<wire x1="12" y1="9" x2="8.405" y2="12.595" width="0.8128" layer="1"/>
-<wire x1="8.405" y1="12.595" x2="8.405" y2="15.325" width="0.8128" layer="1"/>
+<wire x1="12" y1="9" x2="10" y2="11" width="0.8128" layer="1"/>
+<wire x1="10" y1="11" x2="6" y2="11" width="0.8128" layer="1"/>
+<wire x1="6" y1="11" x2="4" y2="13" width="0.8128" layer="1"/>
+<wire x1="4" y1="13" x2="4" y2="18" width="0.8128" layer="1"/>
+<wire x1="4" y1="18" x2="5.425" y2="19.425" width="0.8128" layer="1"/>
+<wire x1="5.425" y1="19.425" x2="8.405" y2="19.425" width="0.8128" layer="1"/>
 </signal>
 <signal name="SIG1_2_NC">
 <contactref element="J3" pad="1"/>
-<contactref element="K1" pad="5"/>
-<wire x1="8.405" y1="19.425" x2="11.575" y2="19.425" width="0.8128" layer="1"/>
-<wire x1="11.575" y1="19.425" x2="14.54" y2="16.46" width="0.8128" layer="1"/>
-<wire x1="14.54" y1="16.46" x2="14.54" y2="5" width="0.8128" layer="1"/>
+<contactref element="K1" pad="1"/>
+<wire x1="8.405" y1="15.325" x2="12.675" y2="15.325" width="0.8128" layer="1"/>
+<wire x1="12.675" y1="15.325" x2="14.54" y2="13.46" width="0.8128" layer="1"/>
+<wire x1="14.54" y1="13.46" x2="14.54" y2="5" width="0.8128" layer="1"/>
 </signal>
 <signal name="SIG3_1_NC">
 <contactref element="J8" pad="1"/>
-<contactref element="K3" pad="8"/>
-<wire x1="70.54" y1="5" x2="70.54" y2="10.54" width="0.8128" layer="1"/>
-<wire x1="70.54" y1="10.54" x2="74" y2="14" width="0.8128" layer="1"/>
-<wire x1="74" y1="14" x2="74" y2="18" width="0.8128" layer="1"/>
-<wire x1="74" y1="18" x2="72.575" y2="19.425" width="0.8128" layer="1"/>
-<wire x1="72.575" y1="19.425" x2="70.605" y2="19.425" width="0.8128" layer="1"/>
+<contactref element="K3" pad="4"/>
+<wire x1="70.54" y1="5" x2="70.605" y2="5.065" width="0.8128" layer="1"/>
+<wire x1="70.605" y1="5.065" x2="70.605" y2="15.325" width="0.8128" layer="1"/>
 </signal>
 <signal name="SIG3_1_NO">
 <contactref element="J8" pad="2"/>
-<contactref element="K3" pad="4"/>
+<contactref element="K3" pad="8"/>
 <wire x1="68" y1="5" x2="68" y2="14" width="0.8128" layer="1"/>
-<wire x1="68" y1="14" x2="69.325" y2="15.325" width="0.8128" layer="1"/>
-<wire x1="69.325" y1="15.325" x2="70.605" y2="15.325" width="0.8128" layer="1"/>
+<wire x1="68" y1="14" x2="67" y2="15" width="0.8128" layer="1"/>
+<wire x1="67" y1="15" x2="67" y2="17" width="0.8128" layer="1"/>
+<wire x1="67" y1="17" x2="69.425" y2="19.425" width="0.8128" layer="1"/>
+<wire x1="69.425" y1="19.425" x2="70.605" y2="19.425" width="0.8128" layer="1"/>
 </signal>
 <signal name="SIG3_2_NC">
 <contactref element="J9" pad="1"/>
-<contactref element="K3" pad="5"/>
-<wire x1="61.54" y1="5" x2="61.54" y2="17.46" width="0.8128" layer="1"/>
-<wire x1="61.54" y1="17.46" x2="59.575" y2="19.425" width="0.8128" layer="1"/>
-<wire x1="59.575" y1="19.425" x2="57.405" y2="19.425" width="0.8128" layer="1"/>
+<contactref element="K3" pad="1"/>
+<wire x1="61.54" y1="5" x2="61.54" y2="13.46" width="0.8128" layer="1"/>
+<wire x1="61.54" y1="13.46" x2="59.675" y2="15.325" width="0.8128" layer="1"/>
+<wire x1="59.675" y1="15.325" x2="57.405" y2="15.325" width="0.8128" layer="1"/>
 </signal>
 <signal name="SIG3_2_NO">
 <contactref element="J9" pad="2"/>
-<contactref element="K3" pad="1"/>
-<wire x1="59" y1="5" x2="59" y2="11" width="0.8128" layer="1"/>
-<wire x1="59" y1="11" x2="57.405" y2="12.595" width="0.8128" layer="1"/>
-<wire x1="57.405" y1="12.595" x2="57.405" y2="15.325" width="0.8128" layer="1"/>
+<contactref element="K3" pad="5"/>
+<wire x1="59" y1="5" x2="59" y2="10" width="0.8128" layer="1"/>
+<wire x1="59" y1="10" x2="58" y2="11" width="0.8128" layer="1"/>
+<wire x1="58" y1="11" x2="54" y2="11" width="0.8128" layer="1"/>
+<wire x1="54" y1="11" x2="53" y2="12" width="0.8128" layer="1"/>
+<wire x1="53" y1="12" x2="53" y2="18" width="0.8128" layer="1"/>
+<wire x1="53" y1="18" x2="54.425" y2="19.425" width="0.8128" layer="1"/>
+<wire x1="54.425" y1="19.425" x2="57.405" y2="19.425" width="0.8128" layer="1"/>
 </signal>
 <signal name="SIG_IN_3">
