File: EXM Relay Three/Rev A1/EXM Relay Three - Rev A1.sch (EAGLE design)
At the start: 23 parts, among them J1 MSTBA3, J10 MSTBA2, J2 MSTBA3, J3 22-05-7038-03, J4 22-05-7038-03, J5 22-05-7038-03, J6 22-05-7038-03, J7 MSTBA3, J8 22-05-7038-03, J9 22-05-7038-03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

Commit message: Renumber outputs and change silkscreen
Connections:
- net SIG1_1_NC: now also J3-1.S, K1G$3.NC; no longer J4-1.S, K1G$2.NC
- net SIG1_1_NO: now also J3-2.S, K1G$3.NO; no longer J4-2.S, K1G$2.NO
- net SIG1_2_NC: now also J4-1.S, K1G$2.NC; no longer J3-1.S, K1G$3.NC
- net SIG1_2_NO: now also J4-2.S, K1G$2.NO; no longer J3-2.S, K1G$3.NO
- net SIG2_1_NC: now also J6-1.S, K2G$3.NC; no longer J5-1.S, K2G$2.NC
- net SIG2_1_NO: now also J6-2.S, K2G$3.NO; no longer J5-2.S, K2G$2.NO
- net SIG2_2_NC: now also J5-1.S, K2G$2.NC; no longer J6-1.S, K2G$3.NC
- net SIG2_2_NO: now also J5-2.S, K2G$2.NO; no longer J6-2.S, K2G$3.NO
- net SIG3_1_NC: now also J9-1.S, K3G$3.NC; no longer J8-1.S, K3G$2.NC
- net SIG3_1_NO: now also J9-2.S, K3G$3.NO; no longer J8-2.S, K3G$2.NO
- net SIG3_2_NC: now also J8-1.S, K3G$2.NC; no longer J9-1.S, K3G$3.NC
- net SIG3_2_NO: now also J8-2.S, K3G$2.NO; no longer J9-2.S, K3G$3.NO
Changed lines of the file:
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@@
 </segment>
 </net>
-<net name="SIG2_1_NO" class="0">
-<segment>
-<wire x1="27.94" y1="170.18" x2="38.1" y2="170.18" width="0.1524" layer="91"/>
-<label x="38.1" y="170.18" size="1.27" layer="95" xref="yes"/>
-<pinref part="J5" gate="-2" pin="S"/>
-</segment>
-<segment>
-<wire x1="167.64" y1="144.78" x2="177.8" y2="144.78" width="0.1524" layer="91"/>
-<label x="177.8" y="144.78" size="1.27" layer="95" xref="yes"/>
-<pinref part="K2" gate="G$2" pin="NO"/>
-<wire x1="167.64" y1="147.32" x2="167.64" y2="144.78" width="0.1524" layer="91"/>
-</segment>
-</net>
-<net name="SIG1_1_NC" class="0">
+<net name="SIG1_2_NC" class="0">
 <segment>
 <pinref part="J4" gate="-1" pin="S"/>
@@
 </segment>
 </net>
-<net name="SIG2_2_NC" class="0">
+<net name="SIG2_1_NC" class="0">
 <segment>
 <wire x1="167.64" y1="137.16" x2="177.8" y2="137.16" width="0.1524" layer="91"/>
@@
 </segment>
 </net>
-<net name="SIG2_2_NO" class="0">
+<net name="SIG2_1_NO" class="0">
 <segment>
 <wire x1="167.64" y1="121.92" x2="177.8" y2="121.92" width="0.1524" layer="91"/>
@@
 </segment>
 </net>
-<net name="SIG2_1_NC" class="0">
+<net name="SIG2_2_NC" class="0">
 <segment>
 <pinref part="J5" gate="-1" pin="S"/>
@@
 </segment>
 </net>
-<net name="SIG1_1_NO" class="0">
+<net name="SIG1_2_NO" class="0">
 <segment>
 <wire x1="167.64" y1="210.82" x2="177.8" y2="210.82" width="0.1524" layer="91"/>
@@
 </segment>
 </net>
-<net name="SIG1_2_NO" class="0">
+<net name="SIG1_1_NO" class="0">
 <segment>
 <pinref part="J3" gate="-2" pin="S"/>
@@
 </segment>
 </net>
-<net name="SIG1_2_NC" class="0">
+<net name="SIG1_1_NC" class="0">
 <segment>
 <pinref part="J3" gate="-1" pin="S"/>
@@
 </segment>
 </net>
-<net name="SIG3_1_NC" class="0">
+<net name="SIG3_2_NC" class="0">
 <segment>
 <pinref part="J8" gate="-1" pin="S"/>
@@
 </segment>
 </net>
-<net name="SIG3_1_NO" class="0">
+<net name="SIG3_2_NO" class="0">
 <segment>
 <wire x1="27.94" y1="104.14" x2="38.1" y2="104.14" width="0.1524" layer="91"/>
@@
 </segment>
 </net>
-<net name="SIG3_2_NC" class="0">
+<net name="SIG3_1_NC" class="0">
 <segment>
 <pinref part="J9" gate="-1" pin="S"/>
@@
 </segment>
 </net>
-<net name="SIG3_2_NO" class="0">
+<net name="SIG3_1_NO" class="0">
 <segment>
 <pinref part="J9" gate="-2" pin="S"/>
@@
 </segment>
 </net>
+<net name="SIG2_2_NO" class="0">
+<segment>
+<wire x1="167.64" y1="144.78" x2="177.8" y2="144.78" width="0.1524" layer="91"/>
+<label x="177.8" y="144.78" size="1.27" layer="95" xref="yes"/>
+<pinref part="K2" gate="G$2" pin="NO"/>
+<wire x1="167.64" y1="147.32" x2="167.64" y2="144.78" width="0.1524" layer="91"/>
+</segment>
+<segment>
+<wire x1="27.94" y1="170.18" x2="38.1" y2="170.18" width="0.1524" layer="91"/>
+<label x="38.1" y="170.18" size="1.27" layer="95" xref="yes"/>
+<pinref part="J5" gate="-2" pin="S"/>
+</segment>
+</net>

Commit message: Generate MDP files
Parts:
- CC1, JP1, JP2, JP3, JP4, MP1, MP2, MP3, MP4, T1: OC_NEWARK (none) -> unknown
- J2: value MSTBA3 -> 22-05-7038-03; device con-phoenix-508:MSTBA3 -> con-molex:22-05-7038-03; MPN (none) -> 22-05-7038; OC_NEWARK (none) -> 26M6362
- J3, J5, J6, J8, J9: MPN (none) -> 22-05-7038; OC_NEWARK (none) -> 26M6362
- J4: value 22-05-7038-03 -> MSTBA3; device con-molex:22-05-7038-03 -> con-phoenix-508:MSTBA3
- K1, K2, K3: MF (none) -> OMRON COMPONENTS USA; MPN (none) -> MY2-02-DC24; OC_NEWARK (none) -> 96B2719
Connections:
- net +24V: now also J4-1.1; no longer J2-1.1
- net GND: now also J2-3.S, J4-3.1; no longer J2-3.1, J4-3.S
- net SIG1_1_NC: now also J9-1.S, K3G$3.NC; no longer J3-1.S, K1G$3.NC
- net SIG1_1_NO: now also J9-2.S, K3G$3.NO; no longer J3-2.S, K1G$3.NO
- net SIG1_2_NC: now also J8-1.S, K3G$2.NC; no longer J4-1.S, K1G$2.NC
- net SIG1_2_NO: now also J8-2.S, K3G$2.NO; no longer J4-2.S, K1G$2.NO
- net SIG3_1_NC: now also J3-1.S, K1G$3.NC; no longer J9-1.S, K3G$3.NC
- net SIG3_1_NO: now also J3-2.S, K1G$3.NO; no longer J9-2.S, K3G$3.NO
- net SIG3_2_NC: now also J2-1.S, K1G$2.NC; no longer J8-1.S, K3G$2.NC
- net SIG3_2_NO: now also J2-2.S, K1G$2.NO; no longer J8-2.S, K3G$2.NO
- net SIG_IN_1: now also J7-2.1, K3G$1.+; no longer J2-2.1, K1G$1.+
- net SIG_IN_2: now also J4-2.1; no longer J1-2.1
- net SIG_IN_3: now also J1-2.1, K1G$1.+; no longer J7-2.1, K3G$1.+
Other:
- moved on the sheet: J1-1, J1-2, J1-3, J3-1, J3-2, J3-3, J7-1, J7-2, J7-3, J8-1, J8-2, J8-3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

Commit message: Generated BOM files
Parts:
- K1, K2, K3: MPN MY2-02-DC24 -> PY08; OC_NEWARK 96B2719 -> 36K3464
Changed lines of the file:
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@@
 <part name="K3" library="rel-omron" deviceset="MY2" device="">
 <attribute name="MF" value="OMRON COMPONENTS USA"/>
-<attribute name="MPN" value="MY2-02-DC24"/>
-<attribute name="OC_NEWARK" value="96B2719"/>
+<attribute name="MPN" value="PY08"/>
+<attribute name="OC_NEWARK" value="36K3464"/>
 </part>
 <part name="P+5" library="supply3" deviceset="+24V" device=""/>
@@
 <part name="K2" library="rel-omron" deviceset="MY2" device="">
 <attribute name="MF" value="OMRON COMPONENTS USA"/>
-<attribute name="MPN" value="MY2-02-DC24"/>
-<attribute name="OC_NEWARK" value="96B2719"/>
+<attribute name="MPN" value="PY08"/>
+<attribute name="OC_NEWARK" value="36K3464"/>
 </part>
 <part name="P+3" library="supply3" deviceset="+24V" device=""/>
@@
 <part name="K1" library="rel-omron" deviceset="MY2" device="">
 <attribute name="MF" value="OMRON COMPONENTS USA"/>
-<attribute name="MPN" value="MY2-02-DC24"/>
-<attribute name="OC_NEWARK" value="96B2719"/>
+<attribute name="MPN" value="PY08"/>
+<attribute name="OC_NEWARK" value="36K3464"/>
 </part>
 <part name="P+1" library="supply3" deviceset="+24V" device=""/>
