File: EXM Relay Three/Rev A2/EXM Relay Three - Rev A2.sch (EAGLE design)
At the start: 23 parts, among them J1 22-05-7048-04, J10 MSTBA3, J2 22-05-7048-04, J3 MSTBA3, J4 22-05-7048-04, J5 22-05-7048-04, J6 MSTBA3, J7 22-05-7048-04, J8 22-05-7048-04, J9 MSTBA2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

Commit message: Renumber part and updated BOM
Parts:
- J10: value MSTBA3 -> MSTBA2; device con-phoenix-508:MSTBA3 -> con-phoenix-508:MSTBA2
- J9: value MSTBA2 -> MSTBA3; device con-phoenix-508:MSTBA2 -> con-phoenix-508:MSTBA3
Connections:
- net GND: now also J10-2.1, J9-3.1; no longer J10-3.1, J9-2.1
- net SIG3_1_C: now also J7-1.S; no longer J8-1.S
- net SIG3_1_NC: now also J7-2.S; no longer J8-2.S
- net SIG3_1_NO: now also J7-3.S; no longer J8-3.S
- net SIG3_2_C: now also J8-1.S; no longer J7-1.S
- net SIG3_2_NC: now also J8-2.S; no longer J7-2.S
- net SIG3_2_NO: now also J8-3.S; no longer J7-3.S
- net SIG_IN_3: now also J9-2.1; no longer J10-2.1
Other:
- moved on the sheet: J10-1, J10-2, J7-1, J7-2, J7-3, J7-4, J8-1, J8-2, J8-3, J8-4, J9-1, J9-2
Changed lines of the file:
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@@
 <part name="GND7" library="supply3" deviceset="GND" device=""/>
 <part name="GND5" library="supply3" deviceset="GND" device=""/>
-<part name="J10" library="con-phoenix-508" deviceset="MSTBA3" device=""/>
+<part name="J9" library="con-phoenix-508" deviceset="MSTBA3" device=""/>
 <part name="K3" library="rel-omron" deviceset="MY2" device="">
 <attribute name="MF" value="OMRON COMPONENTS USA"/>
@@
 <attribute name="OC_NEWARK" value="36K3464"/>
 </part>
-<part name="P+4" library="supply3" deviceset="+24V" device=""/>
-<part name="GND13" library="supply3" deviceset="GND" device=""/>
-<part name="GND9" library="supply3" deviceset="GND" device=""/>
+<part name="P+3" library="supply3" deviceset="+24V" device=""/>
 <part name="GND12" library="supply3" deviceset="GND" device=""/>
 <part name="GND10" library="supply3" deviceset="GND" device=""/>
-<part name="J9" library="con-phoenix-508" deviceset="MSTBA2" device=""/>
 <part name="GND11" library="supply3" deviceset="GND" device=""/>
-<part name="P+3" library="supply3" deviceset="+24V" device=""/>
+<part name="GND9" library="supply3" deviceset="GND" device=""/>
+<part name="J10" library="con-phoenix-508" deviceset="MSTBA2" device=""/>
+<part name="GND13" library="supply3" deviceset="GND" device=""/>
+<part name="P+4" library="supply3" deviceset="+24V" device=""/>
 <part name="JP1" library="SparkFun" deviceset="FIDUCIAL" device="1X2">
 <attribute name="MF" value=""/>
@@
 <part name="J5" library="con-molex" deviceset="22-?-04" device="05-7048"/>
 <part name="J4" library="con-molex" deviceset="22-?-04" device="05-7048"/>
+<part name="J8" library="con-molex" deviceset="22-?-04" device="05-7048"/>
 <part name="J7" library="con-molex" deviceset="22-?-04" device="05-7048"/>
-<part name="J8" library="con-molex" deviceset="22-?-04" device="05-7048"/>
 </parts>
 <sheets>
@@
 <instance part="K2" gate="G$3" x="170.18" y="167.64" rot="MR90"/>
 <instance part="GND5" gate="1" x="38.1" y="162.56"/>
-<instance part="J10" gate="-1" x="25.4" y="50.8"/>
-<instance part="J10" gate="-2" x="25.4" y="45.72"/>
-<instance part="J10" gate="-3" x="25.4" y="40.64"/>
+<instance part="J9" gate="-1" x="25.4" y="50.8"/>
+<instance part="J9" gate="-2" x="25.4" y="45.72"/>
+<instance part="J9" gate="-3" x="25.4" y="40.64"/>
 <instance part="K3" gate="G$2" x="170.18" y="48.26" rot="MR90">
 <attribute name="OC_NEWARK" x="170.18" y="48.26" size="1.778" layer="96" display="off"/>
@@
 </instance>
 <instance part="K3" gate="G$1" x="137.16" y="60.96"/>
-<instance part="P+4" gate="1" x="35.56" y="58.42"/>
-<instance part="GND13" gate="1" x="35.56" y="35.56"/>
-<instance part="GND9" gate="1" x="86.36" y="68.58"/>
-<instance part="GND12" gate="1" x="137.16" y="48.26"/>
+<instance part="P+3" gate="1" x="35.56" y="58.42"/>
+<instance part="GND12" gate="1" x="35.56" y="35.56"/>
+<instance part="GND10" gate="1" x="86.36" y="68.58"/>
+<instance part="GND11" gate="1" x="137.16" y="48.26"/>
 <instance part="K3" gate="G$3" x="170.18" y="71.12" rot="MR90"/>
-<instance part="GND10" gate="1" x="38.1" y="68.58"/>
-<instance part="J9" gate="-1" x="360.68" y="63.5"/>
-<instance part="J9" gate="-2" x="360.68" y="58.42"/>
-<instance part="GND11" gate="1" x="370.84" y="50.8"/>
-<instance part="P+3" gate="1" x="370.84" y="71.12"/>
+<instance part="GND9" gate="1" x="38.1" y="68.58"/>
+<instance part="J10" gate="-1" x="360.68" y="243.84"/>
+<instance part="J10" gate="-2" x="360.68" y="238.76"/>
+<instance part="GND13" gate="1" x="370.84" y="231.14"/>
+<instance part="P+4" gate="1" x="370.84" y="251.46"/>
 <instance part="JP1" gate="G$1" x="345.44" y="22.86">
 <attribute name="OC_NEWARK" x="345.44" y="22.86" size="1.778" layer="96" display="off"/>
@@
 <instance part="J4" gate="-3" x="25.4" y="170.18" rot="MR0"/>
 <instance part="J4" gate="-4" x="25.4" y="165.1" rot="MR0"/>
-<instance part="J7" gate="-1" x="76.2" y="86.36" rot="MR0"/>
-<instance part="J7" gate="-2" x="76.2" y="81.28" rot="MR0"/>
-<instance part="J7" gate="-3" x="76.2" y="76.2" rot="MR0"/>
-<instance part="J7" gate="-4" x="76.2" y="71.12" rot="MR0"/>
-<instance part="J8" gate="-1" x="25.4" y="86.36" rot="MR0"/>
-<instance part="J8" gate="-2" x="25.4" y="81.28" rot="MR0"/>
-<instance part="J8" gate="-3" x="25.4" y="76.2" rot="MR0"/>
-<instance part="J8" gate="-4" x="25.4" y="71.12" rot="MR0"/>
+<instance part="J8" gate="-1" x="76.2" y="86.36" rot="MR0"/>
+<instance part="J8" gate="-2" x="76.2" y="81.28" rot="MR0"/>
+<instance part="J8" gate="-3" x="76.2" y="76.2" rot="MR0"/>
+<instance part="J8" gate="-4" x="76.2" y="71.12" rot="MR0"/>
+<instance part="J7" gate="-1" x="25.4" y="86.36" rot="MR0"/>
+<instance part="J7" gate="-2" x="25.4" y="81.28" rot="MR0"/>
+<instance part="J7" gate="-3" x="25.4" y="76.2" rot="MR0"/>
+<instance part="J7" gate="-4" x="25.4" y="71.12" rot="MR0"/>
 </instances>
 <busses>
@@
 </segment>
 <segment>
+<pinref part="J9" gate="-1" pin="1"/>
+<pinref part="P+3" gate="1" pin="+24V"/>
+<wire x1="30.48" y1="50.8" x2="35.56" y2="50.8" width="0.1524" layer="91"/>
+<wire x1="35.56" y1="50.8" x2="35.56" y2="55.88" width="0.1524" layer="91"/>
+</segment>
+<segment>
 <pinref part="J10" gate="-1" pin="1"/>
 <pinref part="P+4" gate="1" pin="+24V"/>
-<wire x1="30.48" y1="50.8" x2="35.56" y2="50.8" width="0.1524" layer="91"/>
-<wire x1="35.56" y1="50.8" x2="35.56" y2="55.88" width="0.1524" layer="91"/>
-</segment>
-<segment>
-<pinref part="J9" gate="-1" pin="1"/>
-<pinref part="P+3" gate="1" pin="+24V"/>
-<wire x1="365.76" y1="63.5" x2="370.84" y2="63.5" width="0.1524" layer="91"/>
-<wire x1="370.84" y1="63.5" x2="370.84" y2="68.58" width="0.1524" layer="91"/>
+<wire x1="365.76" y1="243.84" x2="370.84" y2="243.84" width="0.1524" layer="91"/>
+<wire x1="370.84" y1="243.84" x2="370.84" y2="248.92" width="0.1524" layer="91"/>
 </segment>
 </net>
@@
 </segment>
 <segment>
-<pinref part="J10" gate="-3" pin="1"/>
-<pinref part="GND13" gate="1" pin="GND"/>
+<pinref part="J9" gate="-3" pin="1"/>
+<pinref part="GND12" gate="1" pin="GND"/>
 <wire x1="30.48" y1="40.64" x2="35.56" y2="40.64" width="0.1524" layer="91"/>
 <wire x1="35.56" y1="40.64" x2="35.56" y2="38.1" width="0.1524" layer="91"/>
 </segment>
 <segment>
+<pinref part="GND10" gate="1" pin="GND"/>
+<wire x1="78.74" y1="71.12" x2="86.36" y2="71.12" width="0.1524" layer="91"/>
+<pinref part="J8" gate="-4" pin="S"/>
+</segment>
+<segment>
+<pinref part="K3" gate="G$1" pin="-"/>
+<pinref part="GND11" gate="1" pin="GND"/>
+<wire x1="137.16" y1="55.88" x2="137.16" y2="50.8" width="0.1524" layer="91"/>
+</segment>
+<segment>
+<wire x1="27.94" y1="71.12" x2="38.1" y2="71.12" width="0.1524" layer="91"/>
 <pinref part="GND9" gate="1" pin="GND"/>
-<wire x1="78.74" y1="71.12" x2="86.36" y2="71.12" width="0.1524" layer="91"/>
 <pinref part="J7" gate="-4" pin="S"/>
 </segment>
 <segment>
-<pinref part="K3" gate="G$1" pin="-"/>
-<pinref part="GND12" gate="1" pin="GND"/>
-<wire x1="137.16" y1="55.88" x2="137.16" y2="50.8" width="0.1524" layer="91"/>
-</segment>
-<segment>
-<wire x1="27.94" y1="71.12" x2="38.1" y2="71.12" width="0.1524" layer="91"/>
-<pinref part="GND10" gate="1" pin="GND"/>
-<pinref part="J8" gate="-4" pin="S"/>
-</segment>
-<segment>
-<pinref part="J9" gate="-2" pin="1"/>
-<pinref part="GND11" gate="1" pin="GND"/>
-<wire x1="365.76" y1="58.42" x2="370.84" y2="58.42" width="0.1524" layer="91"/>
-<wire x1="370.84" y1="58.42" x2="370.84" y2="53.34" width="0.1524" layer="91"/>
+<pinref part="J10" gate="-2" pin="1"/>
+<pinref part="GND13" gate="1" pin="GND"/>
+<wire x1="365.76" y1="238.76" x2="370.84" y2="238.76" width="0.1524" layer="91"/>
+<wire x1="370.84" y1="238.76" x2="370.84" y2="233.68" width="0.1524" layer="91"/>
 </segment>
 </net>
@@
 <wire x1="78.74" y1="81.28" x2="88.9" y2="81.28" width="0.1524" layer="91"/>
 <label x="88.9" y="81.28" size="1.27" layer="95" xref="yes"/>
-<pinref part="J7" gate="-2" pin="S"/>
+<pinref part="J8" gate="-2" pin="S"/>
 </segment>
 <segment>
@@
 <wire x1="78.74" y1="76.2" x2="88.9" y2="76.2" width="0.1524" layer="91"/>
 <label x="88.9" y="76.2" size="1.27" layer="95" xref="yes"/>
-<pinref part="J7" gate="-3" pin="S"/>
+<pinref part="J8" gate="-3" pin="S"/>
 </segment>
 <segment>
@@
 <wire x1="27.94" y1="81.28" x2="38.1" y2="81.28" width="0.1524" layer="91"/>
 <label x="38.1" y="81.28" size="1.27" layer="95" xref="yes"/>
-<pinref part="J8" gate="-2" pin="S"/>
+<pinref part="J7" gate="-2" pin="S"/>
 </segment>
 <segment>
@@
 <wire x1="27.94" y1="76.2" x2="38.1" y2="76.2" width="0.1524" layer="91"/>
 <label x="38.1" y="76.2" size="1.27" layer="95" xref="yes"/>
-<pinref part="J8" gate="-3" pin="S"/>
+<pinref part="J7" gate="-3" pin="S"/>
 </segment>
 <segment>
@@
 <net name="SIG_IN_3" class="0">
 <segment>
-<pinref part="J10" gate="-2" pin="1"/>
+<pinref part="J9" gate="-2" pin="1"/>
 <wire x1="30.48" y1="45.72" x2="38.1" y2="45.72" width="0.1524" layer="91"/>
 <label x="38.1" y="45.72" size="1.27" layer="95" xref="yes"/>
@@
 <segment>
 <label x="88.9" y="86.36" size="1.27" layer="95" font="vector" xref="yes"/>
-<pinref part="J7" gate="-1" pin="S"/>
+<pinref part="J8" gate="-1" pin="S"/>
 <wire x1="78.74" y1="86.36" x2="88.9" y2="86.36" width="0.1524" layer="91"/>
 </segment>
@@
 <segment>
 <label x="38.1" y="86.36" size="1.27" layer="95" font="vector" xref="yes"/>
-<pinref part="J8" gate="-1" pin="S"/>
+<pinref part="J7" gate="-1" pin="S"/>
 <wire x1="27.94" y1="86.36" x2="38.1" y2="86.36" width="0.1524" layer="91"/>
 </segment>
