File: EXM Encoder/Rev A1/EXM Encoder - Rev A1.brd (EAGLE design)
At the start: 160 x 100 mm, 8 parts, among them J2 22-05-7058-05, T1 EXMACHINA-LOGO-NAME

Commit message: Route the board
Parts:
- moved J2 73.0 mm to (15.0, 5.00)
- moved JP3 64.5 mm to (28.0, 2.00)
- moved E1 62.1 mm to (15.0, 23.0)
- moved JP4 61.1 mm to (28.0, 33.0)
- moved CC1 50.0 mm to (26.5, 9.95), turned to 90 degrees
- moved JP1 38.6 mm to (2.00, 2.00)
- moved T1 37.4 mm to (4.10, 6.06), turned to 90 degrees
- moved JP2 30.2 mm to (2.00, 33.0)
Routing:
- net ENCODER_PUSH: track 0.00 -> 11.0 mm
- net ENCODER_B: track 0.00 -> 8.52 mm
- net ENCODER_A: track 0.00 -> 8.50 mm
- added copper zone on layer 1, net GND
- added copper zone on layer 16, net GND
Other:
- board size 160 x 100 mm -> 30 x 35 mm
- board text added: "+5V"
- board text added: "A"
- board text added: "B"
- board text added: "EXM Encoder Rev A1"
- board text added: "GND"
- board text added: "PUSH"
