File: EXM HMI LED/Rev A1/EXM HMI LED - Rev A1.brd (EAGLE design)
At the start: 75 x 10 mm, 17 parts, among them J1 22-05-7058-05, T1 EXMACHINA-LOGO-NAME

Commit message: Generated MDP files
Parts:
- added U$1: (no value), frames:A4L-LOC
Other:
- board text added: "EXM HMI LED Rev A1"
