File: BPtoJTAG_ISCP/BPtoJTAG_ICSP - Rev A1.brd (EAGLE design)
At the start: 60 x 37 mm, 16 parts, among them J1 22-27-2061-06, J2 FTSH-105-01-L-DV, J3 FTSH-103-01-L-DV, J4 F-2X5, P1 F-2X3, U5 TC1264-3.3

Commit message: Final revision before review:
- Update package silkscreen
- Reroute to prevent GND from being broke
- Change signal trace width to 8mil
- Change power trace width to 12mil
- Connect FTDI +5V to converter instead of VDD
Parts:
- added CC1: CC-BY-NC-SA, cc-by-sa:CC-BY-NC-SA
- added LED1, LED2, LED3: (no value), led:CHIPLED_0603
- added R1, R2, R3: 1K5, rcl:R0603
- added T1: EXMACHINA-LOGO-NAME, exmachina:EXM-LOGO-BASELINE
- MP1, MP2, MP3, MP4: value MOUNT-PAD3,0 -> MOUNT-PAD3.5; device holes:P3,0 -> holes:P3,5
- turned VSEL to 270 degrees
Connections:
- new net N$1: LED1.A, R1.1
- new net N$2: LED2.A, R2.1
- new net N$3: LED3.A, R3.1
- net +3V3: now also R3.2
- net +5V: now also J1.3, R2.2
- net GND: now also LED1.C, LED2.C, LED3.C
- net VDD: no longer J1.3
- net VDD33A1: now also R1.2
Routing:
- net +5V: track 37.2 -> 65.7 mm, vias 1 -> 2
- net VDD: track 78.2 -> 54.5 mm, vias 0 -> 1
- net +3V3: track 22.3 -> 30.7 mm
- net TMS: track 71.5 -> 77.5 mm
- net MOSI: track 98.6 -> 92.6 mm, vias 3 -> 4
- net MISO: track 94.4 -> 98.8 mm
- net TCK/NBOOT: track 102.3 -> 100.4 mm, vias 5 -> 4
- net !RST: track 92.4 -> 94.2 mm, vias 2 -> 3
- net GND: track 7.38 -> 8.89 mm, vias 4 -> 11
- net N$3: track 0.00 -> 1.50 mm
- net N$2: track 0.00 -> 1.50 mm
- net N$1: track 0.00 -> 1.50 mm
- net VDD33A1: track 11.3 -> 10.5 mm
Other:
- board text added: "+3V3"
- board text added: "+5V"
- board text added: "1.27mm"
- board text added: "2.54mm"
- board text added: "BPtoJTAG_ICSP Rev A1"
- board text added: "BPv3"
- board text added: "BPv4"
- board text added: "ICSP"
- board text added: "JTAG"
