File: BPtoJTAG_ISCP/BPtoJTAG_ICSP - Rev A1.sch (EAGLE design)
At the start: 16 parts, among them J1 22-27-2061-06, J2 FTSH-105-01-L-DV, J3 FTSH-103-01-L-DV, J4 F-2X5, P1 F-2X3, U5 TC1264-3.3

Commit message: Final revision before review:
- Update package silkscreen
- Reroute to prevent GND from being broke
- Change signal trace width to 8mil
- Change power trace width to 12mil
- Connect FTDI +5V to converter instead of VDD
Parts:
- added CC1: CC-BY-NC-SA, cc-by-sa:CC-BY-NC-SA
- added LED1, LED2, LED3: (no value), led:LEDCHIPLED_0603
- added R1, R2, R3: 1K5, rcl:R-EU_R0603
- added T1: EXMACHINA-LOGO-NAME, exmachina:EXMACHINA-LOGO-NAME
- MP1, MP2, MP3, MP4: value MOUNT-PAD3,0 -> MOUNT-PAD3.5; device holes:MOUNT-PAD3,0 -> holes:MOUNT-PAD3.5
Connections:
- new net N$1: LED1.A, R1.1
- new net N$2: LED2.A, R2.1
- new net N$3: LED3.A, R3.1
- net +3V3: now also R3.2
- net +5V: now also J1-3.S, R2.2
- net GND: now also LED1.C, LED2.C, LED3.C
- net VDD: no longer J1-3.S
- net VDD33A1: now also R1.2
Other:
- note added: "+5V to +3V3 converter"
- note added: "FTDI RS235 6-pin header"
- note added: "ICSP 1.27mm header"
- note added: "ICSP 2.54mm header TagConnect compatible"
- note added: "JTAG 1.27mm header"
- note added: "JTAG 2.54mm header TagConnect compatible"
- moved on the sheet: BP1, C20, C21, D4, J1-1, J1-2, J1-3, J1-4, J1-5, J1-6, J2-1, J2-10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
