File: EXM Relay One/Rev A3/EXM Relay One - Rev A3.brd (EAGLE design)
At the start: 70 x 30 mm, 10 parts, among them J1 MSTBA2, J2 MSTBA3, J3 22-05-7038-03, J4 22-05-7038-03, K1 MY2, T1 EXMACHINA-LOGO-NAME

Commit message: Add EXM Relay One rev A3
Connections:
- new net SIG1_C: J4.3, K1.12
- new net SIG2_C: J3.3, K1.9
- net +24V: no longer K1.12, K1.9
- net GND: no longer J3.3, J4.3
Routing:
- net SIG1_C: track 0.00 -> 38.8 mm
- net SIG2_C: track 0.00 -> 36.0 mm
- net SIG1_NC: track 21.4 -> 23.8 mm
- net SIG1_NO: track 27.3 -> 29.3 mm
- net SIG2_NO: track 29.9 -> 29.2 mm
Other:
- board text added: "C1"
- board text added: "C2"
Changed lines of the file:
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@@
 <text x="62.3" y="13.7" size="1.016" layer="21" rot="R180" align="center-left">NC2</text>
 <text x="62.3" y="10.9" size="1.016" layer="21" rot="R180" align="center-left">NO2</text>
-<text x="62.3" y="16.4" size="1.016" layer="21" rot="R180" align="center-left">GND</text>
+<text x="62.3" y="16.4" size="1.016" layer="21" rot="R180" align="center-left">C1</text>
 <text x="62.3" y="21.6" size="1.016" layer="21" rot="R180" align="center-left">NC1</text>
 <text x="62.3" y="19" size="1.016" layer="21" rot="R180" align="center-left">NO1</text>
-<text x="62.3" y="8.5" size="1.016" layer="21" rot="R180" align="center-left">GND</text>
+<text x="62.3" y="8.5" size="1.016" layer="21" rot="R180" align="center-left">C2</text>
 <dimension x1="0" y1="3" x2="70" y2="5" x3="35" y3="-8" textsize="1.778" layer="47" dtype="horizontal"/>
 <dimension x1="0" y1="27" x2="15" y2="15" x3="7.5" y3="36" textsize="1.778" layer="47" dtype="horizontal"/>
@@
 <dimension x1="3" y1="0" x2="6" y2="30" x3="-14" y3="15" textsize="1.778" layer="47" dtype="vertical"/>
 <dimension x1="15" y1="15" x2="15" y2="0" x3="-9" y3="7.5" textsize="1.778" layer="47" dtype="vertical"/>
+<text x="62.7" y="13.7" size="1.016" layer="22" rot="MR180" align="center-right">NC2</text>
+<text x="62.7" y="10.9" size="1.016" layer="22" rot="MR180" align="center-right">NO2</text>
+<text x="62.7" y="16.4" size="1.016" layer="22" rot="MR180" align="center-right">C1</text>
+<text x="62.7" y="21.6" size="1.016" layer="22" rot="MR180" align="center-right">NC1</text>
+<text x="62.7" y="19" size="1.016" layer="22" rot="MR180" align="center-right">NO1</text>
+<text x="62.7" y="8.5" size="1.016" layer="22" rot="MR180" align="center-right">C2</text>
+<text x="10.3" y="26.2" size="1.016" layer="22" rot="MR0" align="center-right">+24V</text>
+<text x="10.3" y="21.2" size="1.016" layer="22" rot="MR0" align="center-right">GND</text>
+<text x="10.3" y="8.9" size="1.016" layer="22" rot="MR0" align="center-right">SIG</text>
+<text x="10.3" y="3.9" size="1.016" layer="22" rot="MR0" align="center-right">GND</text>
 </plain>
 <attributes>
@@
 <signal name="+24V">
 <contactref element="J2" pad="1"/>
-<contactref element="K1" pad="12"/>
 <polygon width="0.8128" layer="1" isolate="0.3048">
 <vertex x="-15" y="45"/>
@@
 </polygon>
 <contactref element="J1" pad="1"/>
-<contactref element="K1" pad="9"/>
 </signal>
 <signal name="GND">
@@
 </polygon>
 <contactref element="J1" pad="2"/>
-<contactref element="J4" pad="3"/>
-<contactref element="J3" pad="3"/>
 <contactref element="K1" pad="13"/>
 </signal>
@@
 <contactref element="J4" pad="2"/>
 <contactref element="K1" pad="8"/>
-<wire x1="65" y1="19" x2="51" y2="19" width="0.8128" layer="1"/>
-<wire x1="51" y1="19" x2="50" y2="18" width="0.8128" layer="1"/>
-<wire x1="50" y1="18" x2="43.18" y2="18" width="0.8128" layer="1"/>
-<wire x1="43.18" y1="18" x2="39.575" y2="21.605" width="0.8128" layer="1"/>
+<wire x1="39.575" y1="21.605" x2="42.38" y2="18.8" width="0.8128" layer="1"/>
+<wire x1="42.38" y1="18.8" x2="48.7" y2="18.8" width="0.8128" layer="1"/>
+<wire x1="48.7" y1="18.8" x2="52.1" y2="22.2" width="0.8128" layer="1"/>
+<wire x1="52.1" y1="22.2" x2="57.9" y2="22.2" width="0.8128" layer="1"/>
+<wire x1="57.9" y1="22.2" x2="61.1" y2="19" width="0.8128" layer="1"/>
+<wire x1="61.1" y1="19" x2="65" y2="19" width="0.8128" layer="1"/>
 </signal>
 <signal name="SIG1_NC">
 <contactref element="J4" pad="1"/>
 <contactref element="K1" pad="4"/>
-<wire x1="65" y1="21.54" x2="43.74" y2="21.54" width="0.8128" layer="1"/>
-<wire x1="43.74" y1="21.54" x2="43.675" y2="21.605" width="0.8128" layer="1"/>
+<wire x1="59.3" y1="24.5" x2="46.57" y2="24.5" width="0.8128" layer="1"/>
+<wire x1="46.57" y1="24.5" x2="43.675" y2="21.605" width="0.8128" layer="1"/>
+<wire x1="59.3" y1="24.5" x2="62.26" y2="21.54" width="0.8128" layer="1"/>
+<wire x1="62.26" y1="21.54" x2="65" y2="21.54" width="0.8128" layer="1"/>
 </signal>
 <signal name="SIG2_NC">
 <contactref element="J3" pad="1"/>
-<wire x1="65" y1="13.54" x2="61.3" y2="13.54" width="0.8128" layer="1"/>
 <contactref element="K1" pad="1"/>
-<wire x1="43.675" y1="8.405" x2="56.165" y2="8.405" width="0.8128" layer="1"/>
-<wire x1="56.165" y1="8.405" x2="61.3" y2="13.54" width="0.8128" layer="1"/>
+<wire x1="65" y1="13.54" x2="60.54" y2="13.54" width="0.8128" layer="1"/>
+<wire x1="57.1" y1="10.1" x2="45.37" y2="10.1" width="0.8128" layer="1"/>
+<wire x1="45.37" y1="10.1" x2="43.675" y2="8.405" width="0.8128" layer="1"/>
+<wire x1="57.1" y1="10.1" x2="60.54" y2="13.54" width="0.8128" layer="1"/>
 </signal>
 <signal name="SIG2_NO">
 <contactref element="J3" pad="2"/>
-<wire x1="62" y1="11" x2="65" y2="11" width="0.8128" layer="1"/>
 <contactref element="K1" pad="5"/>
-<wire x1="62" y1="11" x2="56" y2="5" width="0.8128" layer="1"/>
-<wire x1="56" y1="5" x2="42" y2="5" width="0.8128" layer="1"/>
-<wire x1="42" y1="5" x2="39.575" y2="7.425" width="0.8128" layer="1"/>
-<wire x1="39.575" y1="7.425" x2="39.575" y2="8.405" width="0.8128" layer="1"/>
+<wire x1="65" y1="11" x2="61.2" y2="11" width="0.8128" layer="1"/>
+<wire x1="57.8" y1="7.6" x2="47.7" y2="7.6" width="0.8128" layer="1"/>
+<wire x1="47.7" y1="7.6" x2="45.7" y2="5.6" width="0.8128" layer="1"/>
+<wire x1="45.7" y1="5.6" x2="41.68" y2="5.6" width="0.8128" layer="1"/>
+<wire x1="61.2" y1="11" x2="57.8" y2="7.6" width="0.8128" layer="1"/>
+<wire x1="41.68" y1="5.6" x2="39.575" y2="7.705" width="0.8128" layer="1"/>
+<wire x1="39.575" y1="7.705" x2="39.575" y2="8.405" width="0.8128" layer="1"/>
+</signal>
+<signal name="SIG2_C">
+<contactref element="J3" pad="3"/>
+<contactref element="K1" pad="9"/>
+<wire x1="65" y1="8.46" x2="61.86" y2="8.46" width="0.8128" layer="1"/>
+<wire x1="61.86" y1="8.46" x2="58.6" y2="5.2" width="0.8128" layer="1"/>
+<wire x1="38.38" y1="3.3" x2="47.1" y2="3.3" width="0.8128" layer="1"/>
+<wire x1="33.275" y1="8.405" x2="38.38" y2="3.3" width="0.8128" layer="1"/>
+<wire x1="47.1" y1="3.3" x2="49" y2="5.2" width="0.8128" layer="1"/>
+<wire x1="49" y1="5.2" x2="58.6" y2="5.2" width="0.8128" layer="1"/>
+</signal>
+<signal name="SIG1_C">
+<contactref element="J4" pad="3"/>
+<contactref element="K1" pad="12"/>
+<wire x1="65" y1="16.46" x2="60.44" y2="16.46" width="0.8128" layer="1"/>
+<wire x1="49.1" y1="16" x2="36" y2="16" width="0.8128" layer="1"/>
+<wire x1="36" y1="16" x2="33.275" y2="18.725" width="0.8128" layer="1"/>
+<wire x1="33.275" y1="18.725" x2="33.275" y2="21.605" width="0.8128" layer="1"/>
+<wire x1="53" y1="19.9" x2="57" y2="19.9" width="0.8128" layer="1"/>
+<wire x1="49.1" y1="16" x2="53" y2="19.9" width="0.8128" layer="1"/>
+<wire x1="57" y1="19.9" x2="60.44" y2="16.46" width="0.8128" layer="1"/>
 </signal>
 </signals>
