File: Switch-Ethernet/Rev A6/SwitchEthernet - Rev A6.brd (EAGLE design)
At the start: 86 x 90 mm, 122 parts, among them J1 22-05-7028-02, J2 NE8FAV, J3 NE8FAV, J4 DF17(4.0)-20DS-0.5V(57), J5 DF17(4.0)-20DP-0.5V(57), J6 RB1-125BAG1A, T1 H1102FNL, T2 H1102FNL, T3 EXMACHINA-LOGO-NAME, U1 TC1264-3.3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

Commit message: generated MDP files of Ethernet switch rev A6
Parts:
- C26: value 0.1uF -> 0.1uF, DNI
- U4: value AT24C02C-SSHM-B -> AT24C02C-SSHM-B, DNI
